Commit message: asdf

File: building_robot/building_robot.sdf.xacro (robot description, xacro)
@@ -7,32 +7,5 @@
             <real_time_factor>1.0</real_time_factor>
         </physics>
-        <plugin
-            filename="gz-sim-physics-system"
-            name="gz::sim::systems::Physics">
-        </plugin>
-        <plugin
-            filename="gz-sim-user-commands-system"
-            name="gz::sim::systems::UserCommands">
-        </plugin>
-        <plugin
-            filename="gz-sim-scene-broadcaster-system"
-            name="gz::sim::systems::SceneBroadcaster">
-        </plugin>
-        <!-- Moving Forward-->
-        <xacro:macro name="key-trig-pub-plugin" params="key value">
-            <plugin filename="gz-sim-triggered-publisher-system"
-                    name="gz::sim::systems::TriggeredPublisher">
-                <input type="gz.msgs.Int32" topic="/keyboard/keypress">
-                  <match field="data">${key}</match>
-                </input>
-                <output type="gz.msgs.Twist" topic="/cmd_vel">
-                  ${value}
-                </output>
-            </plugin>
-        </xacro:macro>
-        <xacro:key-trig-pub-plugin key="16777234" value="linear: {x: 0.0}, angular: {z: 0.5}" />
-        <xacro:key-trig-pub-plugin key="16777235" value="linear: {x: 0.5}, angular: {z: 0.0}" />
-        <xacro:key-trig-pub-plugin key="16777236" value="linear: {x: 0.0}, angular: {z: -0.5}" />
-        <xacro:key-trig-pub-plugin key="16777237" value="linear: {x: -0.5}, angular: {z: 0.0}" />
+        <xacro:include filename="plugins.sdf.xacro"/>
         <light type="directional" name="sun">
             <cast_shadows>true</cast_shadows>
@@ -48,29 +21,5 @@
             <direction>-0.5 0.1 -0.9</direction>
         </light>
-        <model name="ground_plane">
-            <static>true</static>
-            <link name="link">
-                <collision name="collision">
-                <geometry>
-                    <plane>
-                    <normal>0 0 1</normal>
-                    </plane>
-                </geometry>
-                </collision>
-                <visual name="visual">
-                <geometry>
-                    <plane>
-                    <normal>0 0 1</normal>
-                    <size>100 100</size>
-                    </plane>
-                </geometry>
-                <material>
-                    <ambient>0.8 0.8 0.8 1</ambient>
-                    <diffuse>0.8 0.8 0.8 1</diffuse>
-                    <specular>0.8 0.8 0.8 1</specular>
-                </material>
-                </visual>
-            </link>
-        </model>
+        <xacro:include filename="ground_plane.sdf.xacro"/>
         <xacro:include filename="vehicle_blue.sdf.xacro"/>
     </world>

File: hello_world/gui.sdf.xacro (robot description, xacro)
@@ -11,5 +11,5 @@
             <scene>scene</scene>
             <ambient_light>0.4 0.4 0.4</ambient_light>
-            <background_color>0.8 1.0 0.8</background_color>
+            <background_color>0.8 0.8 0.8</background_color>
             <camera_pose>-6 0 6 0 0.5 0</camera_pose>
             <camera_clip>

File: hello_world/hello_world.sdf.xacro (robot description, xacro)
@@ -6,17 +6,24 @@
             <real_time_factor>1.0</real_time_factor>
         </physics>
-        <plugin
-            filename="gz-sim-physics-system"
-            name="gz::sim::systems::Physics">
-        </plugin>
-        <plugin
-            filename="gz-sim-user-commands-system"
-            name="gz::sim::systems::UserCommands">
-        </plugin>
-        <plugin
-            filename="gz-sim-scene-broadcaster-system"
-            name="gz::sim::systems::SceneBroadcaster">
-        </plugin>
+        <xacro:include filename="plugins.sdf.xacro"/>
         <xacro:include filename="gui.sdf.xacro"/>
+        <light type="directional" name="sun">
+            <cast_shadows>true</cast_shadows>
+            <pose>0 0 10 0 0 0</pose>
+            <diffuse>0.8 0.8 0.8 1</diffuse>
+            <specular>0.2 0.2 0.2 1</specular>
+            <attenuation>
+                <range>1000</range>
+                <constant>0.9</constant>
+                <linear>0.01</linear>
+                <quadratic>0.001</quadratic>
+            </attenuation>
+            <direction>-0.5 0.1 -0.9</direction>
+        </light>
+        <include>
+            <name>Coke0</name>
+            <pose>0 0 1 0 0 0</pose>
+            <uri>https://fuel.gazebosim.org/1.0/OpenRobotics/models/Coke</uri>
+        </include>
     </world>
 </sdf>

Commit message: sensor

File: building_robot/building_robot.sdf.xacro (robot description, xacro)
@@ -21,4 +21,5 @@
             <direction>-0.5 0.1 -0.9</direction>
         </light>
+        <xacro:include filename="wall.sdf.xacro"/>
         <xacro:include filename="ground_plane.sdf.xacro"/>
         <xacro:include filename="vehicle_blue.sdf.xacro"/>

File: building_robot/plugins.sdf.xacro (robot description, xacro)
@@ -13,11 +13,9 @@
         name="gz::sim::systems::SceneBroadcaster">
     </plugin>
-    <!-- Moving Forward-->
-    <xacro:macro name="key-trig-pub-plugin" params="key value">
+    <!-- Moving with key -->
+    <xacro:macro name="trig-pub-vel" params="value *input">
         <plugin filename="gz-sim-triggered-publisher-system"
                 name="gz::sim::systems::TriggeredPublisher">
-            <input type="gz.msgs.Int32" topic="/keyboard/keypress">
-              <match field="data">${key}</match>
-            </input>
+            <xacro:insert_block name="input" />
             <output type="gz.msgs.Twist" topic="/cmd_vel">
               ${value}
@@ -25,7 +23,31 @@
         </plugin>
     </xacro:macro>
-    <xacro:key-trig-pub-plugin key="16777234" value="linear: {x: 0.0}, angular: {z: 0.5}" />
-    <xacro:key-trig-pub-plugin key="16777235" value="linear: {x: 0.5}, angular: {z: 0.0}" />
-    <xacro:key-trig-pub-plugin key="16777236" value="linear: {x: 0.0}, angular: {z: -0.5}" />
-    <xacro:key-trig-pub-plugin key="16777237" value="linear: {x: -0.5}, angular: {z: 0.0}" />
+    <xacro:macro name="key-trig-pub-vel" params="key value">
+        <xacro:trig-pub-vel value="${value}">
+            <input type="gz.msgs.Int32" topic="/keyboard/keypress">
+              <match field="data">${key}</match>
+            </input>
+        </xacro:trig-pub-vel>
+    </xacro:macro>
+    <xacro:trig-pub-vel value="linear: {x: 0.0}, angular: {z: 0.0}">
+        <input type="gz.msgs.Boolean" topic="/wall/touched">
+            <match>data: true</match>
+        </input>
+    </xacro:trig-pub-vel>
+    <xacro:key-trig-pub-vel key="16777234" value="linear: {x: 0.0}, angular: {z: 0.5}" />
+    <xacro:key-trig-pub-vel key="16777235" value="linear: {x: 0.5}, angular: {z: 0.0}" />
+    <xacro:key-trig-pub-vel key="16777236" value="linear: {x: 0.0}, angular: {z: -0.5}" />
+    <xacro:key-trig-pub-vel key="16777237" value="linear: {x: -0.5}, angular: {z: 0.0}" />
+    <!-- Sensors -->
+    <plugin filename="gz-sim-imu-system"
+            name="gz::sim::systems::Imu">
+    </plugin>
+    <plugin filename="gz-sim-contact-system"
+            name="gz::sim::systems::Contact">
+    </plugin>
+    <plugin
+        filename="gz-sim-sensors-system"
+        name="gz::sim::systems::Sensors">
+        <render_engine>ogre2</render_engine>
+    </plugin>
 </sdf>

File: building_robot/vehicle_blue.sdf.xacro (robot description, xacro)
@@ -1,2 +1,3 @@
+<?xml version="1.0" ?>
 <sdf version="1.10" xmlns:xacro="http://ros.org/wiki/xacro">
     <model name="vehicle_blue" canonical_link="chassis">
@@ -17,6 +18,9 @@
         </plugin>
         <pose relative_to="world">0 0 0 0 0 0</pose>
+        <frame name="lidar_frame" attached_to='chassis'>
+            <pose>0.8 0 0.5 0 0 0</pose>
+        </frame>
         <link name="chassis">
-          <pose relative_to="__model__">0.5 0 ${wheel_radius} 0 0 0</pose>
+            <pose relative_to="__model__">0.5 0 ${wheel_radius} 0 0 0</pose>
             <inertial> <!--inertial properties of the link mass, inertia matix-->
                 <mass>1.14395</mass>
@@ -50,5 +54,40 @@
                 </geometry>
             </collision>
+            <sensor name="imu_sensor" type="imu">
+                <always_on>1</always_on>
+                <update_rate>1</update_rate>
+                <visualize>true</visualize>
+                <topic>imu</topic>
+            </sensor>
+            <sensor name='gpu_lidar' type='gpu_lidar'>
+                <pose relative_to='lidar_frame'>0 0 0 0 0 0</pose>
+                <topic>lidar</topic>
+                <update_rate>10</update_rate>
+                <ray>
+                    <scan>
+                        <horizontal>
+                            <samples>640</samples>
+                            <resolution>1</resolution>
+                            <min_angle>-1.396263</min_angle>
+                            <max_angle>1.396263</max_angle>
+                        </horizontal>
+                        <vertical>
+                            <samples>1</samples>
+                            <resolution>0.01</resolution>
+                            <min_angle>0</min_angle>
+                            <max_angle>0</max_angle>
+                        </vertical>
+                    </scan>
+                    <range>
+                        <min>0.08</min>
+                        <max>10.0</max>
+                        <resolution>0.01</resolution>
+                    </range>
+                </ray>
+                <always_on>1</always_on>
+                <visualize>true</visualize>
+            </sensor>
         </link>
+<!-- wheel -->
         <xacro:macro name="wheel" params="prefix x y">
           <link name='${prefix}_wheel'>
@@ -87,5 +126,5 @@
               </collision>
           </link>
-        </xacro:macro> <!-- wheel-->
+        </xacro:macro> <!-- wheel -->
         <xacro:macro name="wheel_joint" params="prefix">
             <joint name='${prefix}_wheel_joint' type='revolute'>
@@ -101,13 +140,13 @@
                 </axis>
             </joint>
-        </xacro:macro>
+        </xacro:macro>  <!-- wheel_joint -->
         <xacro:wheel prefix="left" x="-0.5" y="${(chassis_y+wheel_length)/2}"/>
         <xacro:wheel_joint prefix="left"/>
         <xacro:wheel prefix="right" x="-0.5" y="-${(chassis_y+wheel_length)/2}"/>
         <xacro:wheel_joint prefix="right"/>
+<!-- caster wheel -->
         <frame name="caster_frame" attached_to='chassis'>
             <pose>0.8 0 -${wheel_radius/2} 0 0 0</pose>
         </frame>
-        <!--caster wheel-->
         <link name='caster'>
             <pose relative_to='caster_frame'/>
